Commit message: Update model.urdf

File: robot/model.urdf (robot description, URDF)
Before this commit: robot SimQ, 18 links, 17 joints
Joints:
- joint LFHip_joint: limit lower=-3.14 upper=3.14 effort=0 velocity=0 -> lower=-1.046 upper=1.57 effort=0 velocity=0
- joint LFLower_joint: limit lower=-3.14 upper=3.14 effort=0 velocity=0 -> lower=-2.62 upper=2.62 effort=0 velocity=0
- joint LRHip_joint: axis -1.0 0.0 0.0 -> 1.0 0.0 0.0; limit lower=-3.14 upper=3.14 effort=0 velocity=0 -> lower=-1.046 upper=1.57 effort=0 velocity=0
- joint LRLower_joint: limit lower=-3.14 upper=3.14 effort=0 velocity=0 -> lower=-2.62 upper=2.62 effort=0 velocity=0
- joint RFHip_joint: limit lower=-3.14 upper=3.14 effort=0 velocity=0 -> lower=-1.57 upper=1.046 effort=0 velocity=0
- joint RFLower_joint: axis -2.775557561562891e-17 -1.0000000000000002 1.2246467991474772e-16 -> 2.775557561562891e-17 1.0000000000000002 -1.2246467991474772e-16; limit lower=-3.14 upper=3.14 effort=0 velocity=0 -> lower=-2.62 upper=2.62 effort=0 velocity=0
- joint RRHip_joint: axis -1.0 0.0 0.0 -> 1.0 0.0 0.0; limit lower=-3.14 upper=3.14 effort=0 velocity=0 -> lower=-1.57 upper=1.046 effort=0 velocity=0
- joint RRLower_joint: axis -1.3877787807814452e-16 -1.0000000000000016 4.163336342348132e-17 -> 1.3877787807814452e-16 1.0000000000000016 -4.163336342348132e-17; limit lower=-3.14 upper=3.14 effort=0 velocity=0 -> lower=-2.62 upper=2.62 effort=0 velocity=0
